Commit message: All done except last motor, and need to fine tune

File: urdf/my_robot.urdf (robot description, URDF)
Before this commit: robot testing-robot, 9 links, 8 joints
Joints:
- joint joint_arm_to_wrist: origin xyz=-0.103129016876 -0.011158664703 0 rpy=0 0 0 -> xyz=-0.06 -0.011158664703 0.0075 rpy=0 0 0
- joint joint_wrist_to_gripper_base: origin xyz=0 0 0 rpy=0 0 0 -> xyz=-0.06 0 0 rpy=0 0 0

Commit message: All done except gripper

File: urdf/my_robot.urdf (robot description, URDF)
Before this commit: robot testing-robot, 9 links, 8 joints
Links:
- added link barra1_link; collision mesh filename=package://my_robot_rviz/meshes/Barra1.dae scale=1 1 1; visual mesh filename=package://my_robot_rviz/meshes/Barra1.dae scale=1 1 1
- added link barra2_link; collision mesh filename=package://my_robot_rviz/meshes/Barra2.dae scale=1 1 1; visual mesh filename=package://my_robot_rviz/meshes/Barra2.dae scale=1 1 1
- added link engranaje1_link; collision mesh filename=package://my_robot_rviz/meshes/Engranaje1.dae scale=1 1 1; visual mesh filename=package://my_robot_rviz/meshes/Engranaje1.dae scale=1 1 1
- added link engranaje2_link; collision mesh filename=package://my_robot_rviz/meshes/Engranaje2.dae scale=1 1 1; visual mesh filename=package://my_robot_rviz/meshes/Engranaje2.dae scale=1 1 1
- added link tapapgarra_link; collision mesh filename=package://my_robot_rviz/meshes/Tapapgarra.dae scale=1 1 1; visual mesh filename=package://my_robot_rviz/meshes/Tapapgarra.dae scale=1 1 1
Joints:
- removed joint joint_gripper_finger1
- removed joint joint_gripper_finger2
- added joint joint_barra1_finger1: type fixed, parent barra1_link, child gripper_finger1_link, origin xyz=0 0 0 rpy=0 0 0
- added joint joint_barra2_finger2: type fixed, parent barra2_link, child gripper_finger2_link
- added joint joint_base_barra1: type fixed, parent engranaje1_link, child barra1_link, origin xyz=0 0 0 rpy=0 0 0
- added joint joint_base_barra2: type revolute, parent gripper_base_link, child barra2_link, origin xyz=0 0 0 rpy=0 0 0, axis 0 0 1, limit lower=0 upper=3.14 effort=5 velocity=1
- added joint joint_base_engranaje1: type revolute, parent gripper_base_link, child engranaje1_link, origin xyz=-0.035 0.01 0 rpy=0 0 0, axis 0 0 1, limit lower=-1.57 upper=0 effort=5 velocity=1
- added joint joint_base_engranaje2: type revolute, parent gripper_base_link, child engranaje2_link, origin xyz=0 0 0 rpy=0 0 0, axis 0 0 1, limit lower=0 upper=3.14 effort=5 velocity=1
- added joint joint_base_tapapgarra: type fixed, parent gripper_base_link, child tapapgarra_link, origin xyz=-0.05 0 0 rpy=0 0 0
- added joint joint_engranaje1_finger1: type fixed, parent engranaje1_link, child gripper_finger1_link, origin xyz=0 0 0 rpy=0 0 0
- added joint joint_engranaje2_finger2: type fixed, parent engranaje2_link, child gripper_finger2_link
- joint joint_arm_to_wrist: origin xyz=-0.06 -0.011158664703 0.0075 rpy=0 0 0 -> xyz=-0.06 -0.011158664703 0.02 rpy=0 0 0
- joint joint_base_to_central: origin xyz=0 0 0.093107574462890613232 -> xyz=0 0 0.046553787
- joint joint_central_to_forearm: origin xyz=0 0 0.07 rpy=0 0 0 -> xyz=-0.0075 0 0.06 rpy=0 0 0
- joint joint_forearm_to_arm: origin xyz=0 0 0.13 rpy=0 0 0 -> xyz=0 0 0.12 rpy=0 0 0

Commit message: Engranaje2 fixed

File: urdf/my_robot.urdf (robot description, URDF)
Before this commit: robot testing-robot, 14 links, 15 joints
Joints:
- joint joint_base_engranaje2: origin xyz=0 0 0 rpy=0 0 0 -> xyz=-0.035 -0.01 0 rpy=0 0 0
